File: Iggy_pcb/Iggy.kicad_pcb (KiCad board)
At the start: 2 copper layers, 299.9 x 120 mm, 150 parts, among them J1 SM04B-SRSS-TB(LF)(SN), J2 ISP, SW1 SW_Push, SW10 SW_Push, SW11 SW_Push, SW12 SW_Push, SW13 SW_Push, SW14 SW_Push, SW15 SW_Push, SW16 SW_Push, SW17 SW_Push, SW18 SW_Push, SW19 SW_Push, SW2 SW_Push, SW20 SW_Push, SW21 SW_Push, SW22 SW_Push, SW23 SW_Push, SW24 SW_Push, SW25 SW_Push, SW26 SW_Push, SW27 SW_Push, SW28 SW_Push, SW29 SW_Push, SW3 SW_Push, SW30 SW_Push, SW31 SW_Push, SW32 SW_Push, SW33 SW_Push, SW34 SW_Push, SW35 SW_Push, SW36 SW_Push, SW37 SW_Push, SW38 SW_Push, SW39 SW_Push, SW4 SW_Push, SW40 SW_Push, SW41 SW_Push, SW42 SW_Push, SW43 SW_Push, SW44 SW_Push, SW45 SW_Push, SW46 SW_Push, SW47 SW_Push, SW48 SW_Push, SW49 SW_Push, SW5 SW_Push, SW50 SW_Push, SW51 SW_Push, SW52 SW_Push, SW53 SW_Push, SW54 SW_Push, SW55 SW_Push, SW56 SW_Push, SW57 SW_Push, SW58 SW_Push, SW59 SW_Push, SW6 SW_Push, SW60 SW_Push, SW61 SW_Push, SW62 Rotary_Encoder_Switch, SW63 Rotary_Encoder_Switch, SW64 Rotary_Encoder_Switch, SW65 JOYSTICK_THUMB, SW66 RESET, SW67 BOOT, SW7 SW_Push, SW8 SW_Push, SW9 SW_Push, U1 ATMEGA328-PU, U2 DISPLAY-OLED-128X64-I2C-no-li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, U3 DISPLAY-OLED-128X64-I2C-no-li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, U4 MCP23017_SP, Y1 16MHz

Commit message: cleared up libraries, pcb done
Parts:
- removed SW65: JOYSTICK_THUMB, SparkFun-Electromechanical:JOYSTICK
- added D61: 3.6V, Diode_THT:D_DO-35_SOD27_P7.62mm_Horizontal_no_front, F.Cu at (308.5, 35.4)
- added D62: 3.6V, Diode_THT:D_DO-35_SOD27_P7.62mm_Horizontal_no_front, F.Cu at (308.5, 31.2)
- added G***: LOGO, Artwork:Iggy Skeleton, F.Cu at (122.9, 31.3)
- added R8: 1.5k, Resistor_THT:R_Axial_DIN0204_L3.6mm_D1.6mm_P5.08mm_Horizontal_no_front, F.Cu at (303.6, 37.9)
- C2, C3, C4, C5, C6, C7: footprint Capacitor_THT:C_Disc_D4.3mm_W1.9mm_P5.00mm -> Capacitor_THT:C_Disc_D4.3mm_W1.9mm_P5.00mm_no_front
- D1, D10, D11, D12, D16, D17, D18, D19, D2, D20, D21, D22, D23, D24, D25, D26, D27, D3, D31, D32, D33, D34, D35, D36, D37, D38, D39, D4, D40, D41, D42, D46, D47, D48, D49, D5, D50, D51, D52, D53, D54, D55, D56, D57, D6, D7, D8, D9: footprint Diode_THT:D_DO-35_SOD27_P7.62mm_Horizontal -> Diode_THT:D_DO-35_SOD27_P7.62mm_Horizontal_no_front
- R1, R2: value 22 -> 68; footprint Resistor_THT:R_Axial_DIN0204_L3.6mm_D1.6mm_P5.08mm_Horizontal -> Resistor_THT:R_Axial_DIN0204_L3.6mm_D1.6mm_P5.08mm_Horizontal_no_front
- R3, R4, R5, R6, R7: footprint Resistor_THT:R_Axial_DIN0204_L3.6mm_D1.6mm_P5.08mm_Horizontal -> Resistor_THT:R_Axial_DIN0204_L3.6mm_D1.6mm_P5.08mm_Horizontal_no_front
- U1, U4: footprint Package_DIP:DIP-28_W7.62mm -> Package_DIP:DIP-28_W7.62mm_no_front
- U2, U3: value DISPLAY-OLED-128X64-I2C-no-lines -> DISPLAY-OLED-128X64-I2C
- moved D60 18.3 mm to (299.3, 115.4), turned to 270 degrees
- moved D29 6.34 mm to (280.2, 77.1)
- moved SW52 6.34 mm to (145.3, 117.2)
- moved SW57 6.34 mm to (240.6, 117.2)
- moved SW58 6.34 mm to (269.6, 117.2)
- moved SW59 6.34 mm to (288.6, 117.2)
- moved SW63 6.34 mm to (315.1, 81.6)
- moved C1 6.34 mm to (296.5, 38.6)
- moved D10 6.34 mm to (165.0, 29.0)
- moved D38 6.34 mm to (141.1, 26.5)
- moved D41 6.34 mm to (188.4, 26.5)
- moved D53 6.34 mm to (144.9, 25.2)
- moved D56 6.34 mm to (192.2, 25.2)
- moved J2 6.34 mm to (290.0, 23.7)
- moved LED1 6.34 mm to (306.1, 25.7)
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Connections:
- U1 pad 16: COL12 -> Net-(U1-Pad16)
- U1 pad 17: COL13 -> COL12
- U1 pad 18: COL14 -> COL13
- U1 pad 19: Enc1_B -> COL14
- U1 pad 23: Enc1_A -> Enc1_B
- U1 pad 24: Enc2_A -> Enc1_A
- U1 pad 25: Joystick_V -> Enc2_B
- U1 pad 26: Joystick_H -> Enc2_A
- U1 pad 6: Enc2_B -> Net-(U1-Pad6)
Routing:
- net Joystick_V: track 134.7 -> 0.00 mm
- net Joystick_H: track 124.2 -> 0.00 mm
- net +5V: track 328.6 -> 222.6 mm, vias 1 -> 0
- net Enc1_B: track 65.0 -> 53.5 mm
- net Enc2_B: track 101.3 -> 91.3 mm, vias 2 -> 0
- net ROW3: track 356.3 -> 365.9 mm
- net Net-(D17-Pad2): track 56.5 -> 61.6 mm
- net Net-(D60-Pad2): track 16.0 -> 11.2 mm
- net Net-(D30-Pad2): track 11.2 -> 15.9 mm
- net Net-(D61-Pad1): track 16.9 -> 21.4 mm
- net Enc1_A: track 62.1 -> 57.8 mm
- net COL14: track 147.8 -> 151.9 mm
- net ROW0: track 358.1 -> 354.6 mm, vias 1 -> 4
- net COL13: track 96.4 -> 94.1 mm
- net Enc2_A: track 99.6 -> 97.5 mm
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- added copper zone on F.Cu, net (none)
Other:
- board size 299.9 x 120 mm -> 298.6 x 120.2 mm
- board text added: "D+"
- board text added: "D-"
- board text added: "Gnd"
- board text added: "Iggy v1.0 by Alex M"
- board text added: "JLCJLCJLCJLC"
- board text added: "Vcc"
- board text removed: "Joy H"
- board text removed: "Joy V"
- board text removed: "VCC"
