File: Iggy_pcb/Iggy.sch (KiCad schematic (older format))
At the start: 150 parts, among them J1 SM04B-SRSS-TB(LF)(SN), J2 ISP, SW1 SW_Push, SW10 SW_Push, SW11 SW_Push, SW12 SW_Push, SW13 SW_Push, SW14 SW_Push, SW15 SW_Push, SW16 SW_Push, SW17 SW_Push, SW18 SW_Push, SW19 SW_Push, SW2 SW_Push, SW20 SW_Push, SW21 SW_Push, SW22 SW_Push, SW23 SW_Push, SW24 SW_Push, SW25 SW_Push, SW26 SW_Push, SW27 SW_Push, SW28 SW_Push, SW29 SW_Push, SW3 SW_Push, SW30 SW_Push, SW31 SW_Push, SW32 SW_Push, SW33 SW_Push, SW34 SW_Push, SW35 SW_Push, SW36 SW_Push, SW37 SW_Push, SW38 SW_Push, SW39 SW_Push, SW4 SW_Push, SW40 SW_Push, SW41 SW_Push, SW42 SW_Push, SW43 SW_Push, SW44 SW_Push, SW45 SW_Push, SW46 SW_Push, SW47 SW_Push, SW48 SW_Push, SW49 SW_Push, SW5 SW_Push, SW50 SW_Push, SW51 SW_Push, SW52 SW_Push, SW53 SW_Push, SW54 SW_Push, SW55 SW_Push, SW56 SW_Push, SW57 SW_Push, SW58 SW_Push, SW59 SW_Push, SW6 SW_Push, SW60 SW_Push, SW61 SW_Push, SW62 Rotary_Encoder_Switch, SW63 Rotary_Encoder_Switch, SW64 Rotary_Encoder_Switch, SW65 JOYSTICK_THUMB, SW66 RESET, SW67 BOOT, SW7 SW_Push, SW8 SW_Push, SW9 SW_Push, U1 ATMEGA328-PU, U2 DISPLAY-OLED-128X64-I2C, U3 DISPLAY-OLED-128X64-I2C, U4 MCP23017_SP, Y1 16MHz

Commit message: cleared up libraries, pcb done
Parts:
- removed SW65: JOYSTICK_THUMB, SparkFun-Electromechanical:JOYSTICK, symbol SparkFun-Switches:JOYSTICK_THUMB
- added D61, D62: 3.6V, Diode_THT:D_DO-35_SOD27_P7.62mm_Horizontal, symbol Device:D_Schottky_Small
- added R8: 1.5k, Resistor_THT:R_Axial_DIN0204_L3.6mm_D1.6mm_P5.08mm_Horizontal, symbol Device:R_Small
- C2, C3, C4, C5, C6, C7: footprint Capacitor_THT:C_Disc_D4.3mm_W1.9mm_P5.00mm -> Capacitor_THT:C_Disc_D4.3mm_W1.9mm_P5.00mm_no_front
- D1, D10, D11, D12, D16, D17, D18, D19, D2, D20, D21, D22, D23, D24, D25, D26, D27, D3, D31, D32, D33, D34, D35, D36, D37, D38, D39, D4, D40, D41, D42, D46, D47, D48, D49, D5, D50, D51, D52, D53, D54, D55, D56, D57, D6, D7, D8, D9: footprint Diode_THT:D_DO-35_SOD27_P7.62mm_Horizontal -> Diode_THT:D_DO-35_SOD27_P7.62mm_Horizontal_no_front
- R1, R2: value 22 -> 68; footprint Resistor_THT:R_Axial_DIN0204_L3.6mm_D1.6mm_P5.08mm_Horizontal -> Resistor_THT:R_Axial_DIN0204_L3.6mm_D1.6mm_P5.08mm_Horizontal_no_front
- R3, R6, R7: footprint Resistor_THT:R_Axial_DIN0204_L3.6mm_D1.6mm_P5.08mm_Horizontal -> Resistor_THT:R_Axial_DIN0204_L3.6mm_D1.6mm_P5.08mm_Horizontal_no_front
- U1, U4: footprint Package_DIP:DIP-28_W7.62mm -> Package_DIP:DIP-28_W7.62mm_no_front
Connections:
- net Joystick_H is gone; now on net Enc2_A: U1.26 (PC3)
- net Joystick_V is gone; now on net Enc2_B: U1.25 (PC2)
- net +5V: now also R8.1
- net COL12: now also U1.17 (PB3); no longer U1.16 (PB2)
- net COL13: now also U1.18 (PB4); no longer U1.17 (PB3)
- net COL14: now also U1.19 (PB5); no longer U1.18 (PB4)
- net Enc1_A: now also U1.24 (PC1); no longer U1.23 (PC0)
- net Enc1_B: now also U1.23 (PC0); no longer U1.19 (PB5)
- net Enc2_A: no longer U1.24 (PC1)
- net Enc2_B: no longer U1.6 (PD4)
- net GND: now also D61.2 (A), D62.2 (A)
- net at J1.2, R1.2: now also D61.1 (K), R8.2
- net at J1.3, R2.2: now also D62.1 (K)
- no-connect marks 7 -> 9
Other:
- note added: "OLED Displays"
- moved on the sheet: C1, C2, C3, C4, C5, R1, R2
